File: Hardware/SAMD21_Pro_RF.brd (EAGLE design)
At the start: 44.5 x 30.5 mm, 129 parts, among them J12 JST, J13 U.FL, J7 PTH, J9 External On/Off, Q1 2.5A/30V, U1 MCP73831, U3 RFM95W, U4 ATSAMD21G, U6 3.3V, Y1 32.768kHz

Commit message: latest
Parts:
- added C7: 1.0uF, SparkFun-Capacitors:0603
- added J10, J14: (no value), SparkFun-Connectors:1X01_NO_SILK
- added LED: (no value), SparkFun-Jumpers:SMT-JUMPER_2_NC_TRACE_SILK
- added LOGO3: QWIIC_LOGO_5MM, SparkFun-Aesthetics:QWIIC_5MM
- added U$34, U$64: (no value), buzzard_labels (1):IO3
- added U$56: (no value), buzzard_labels (1):CLK4
- added U$58, U$59: (no value), buzzard_labels (1):SWD2
- added U$66: (no value), buzzard_labels (2):LED0
- U$60: device Labels:QWIIC-TEXT-04 -> buzzard_labels (1):CLK4
- moved U$51 13.3 mm to (40.2, 19.2)
- moved U$60 13.1 mm to (41.5, 6.50), flipped to the bottom, turned to 90 degrees
- moved U$26 4.02 mm to (-33.0, -17.8)
- moved FD2 1.82 mm to (43.7, 26.0)
- moved FD4 1.82 mm to (43.7, 26.0)
- moved C10 0.52 mm to (34.6, 10.9)
Connections:
- new net N$4: C7.2, U4.43
- new net N$5: LED.2, R13.2
- net 3.3V: now also LED.1; no longer R13.2, U4.43
- net GND: now also C7.1
- net SWDCLK: now also J14.1
- net SWDIO: now also J10.1
Routing:
- net SWDCLK: track 13.4 -> 25.9 mm
- net SWDIO: track 14.6 -> 23.5 mm
- net !RST: track 62.9 -> 71.0 mm, vias 8 -> 6
- net 3.3V: track 111.8 -> 104.4 mm
- net N$5: track 0.00 -> 6.81 mm, vias 0 -> 1
- net N$4: track 0.00 -> 2.37 mm
Other:
- outline, holes or cut-outs redrawn
- board text added: "Pete Lewis"
- board text added: "Revised by:"
- board text added: "v11"
- board text removed: "v10"
