File: Hardware/SAMD21_Pro_RF.sch (EAGLE design)
At the start: 66 parts, among them J12 JST, J13 U.FL, J7 PTH, J9 External On/Off, Q1 2.5A/30V, U1 MCP73831, U3 RFM95W, U4 ATSAMD21G, U6 3.3V, Y1 32.768kHz

Commit message: latest
Parts:
- added C7: 1.0uF, SparkFun-Capacitors:1.0UF-0603-16V-10%
- added J10, J14: (no value), SparkFun-Connectors:CONN_01PTH_NO_SILK_YES_STOP
- added LED: JUMPER-SMT_2_NC_TRACE_SILK, SparkFun-Jumpers:JUMPER-SMT_2_NC_TRACE_SILK
- added LOGO3: QWIIC_LOGO_5MM, SparkFun-Aesthetics:QWIIC_LOGO_5MM
Connections:
- new net N$4: C7.2, U4.VDDCORE
- new net N$5: LED.2, R13.2
- net 3.3V: now also LED.1; no longer R13.2, U4.VDDCORE
- net GND: now also C7.1
- net SWDCLK: now also J14.1
- net SWDIO: now also J10.1
Other:
- note added: "Cut jumper to disable LED"
- note added: "Pete Lewis"
- note added: "Revised by:"
- note added: "VCC RANGE: 1.62-3.63V"
- note added: "v11"
- note removed: "v10"
- moved on the sheet: C4, LED1, R13
